File: kicad/template.kicad_pcb (KiCad board)
At the start: 2 copper layers, 84.1 x 61.7 mm, 8 parts, among them J1 Bus_PCI_Express_x1, J6 USB_C_Receptacle_USB2.0_16P, U2 RP2040, U4 W25Q128JVP, U9 MCP25625T-E/ML, X1 ABM8-272-T3

Commit message: refactor libraries
Parts:
- removed S1, S2: TS-1187A-B-A-B, TS-1187A-B-A-B:SW_TS-1187A-B-A-B
- removed U9: MCP25625T-E/ML, MCP25625T_E_ML:QFN28_6X6MC_MCH
- added U1: MCP25625T-E/ML, challenge_template:QFN28_6X6MC_MCH, F.Cu at (140.1, 80.1)
- added Y1: X322516MLB4SI, challenge_template:OSC_X322516MLB4SI, F.Cu at (127.0, 81.1)
- X1: footprint ABM8-272-T3:ABM8-272-T3_ABR -> challenge_template:ABM8-272-T3_ABR
- moved X1 14.6 mm to (136.8, 96.0)
Connections:
- U4 pad 4: GND -> unconnected-(U4-GND-Pad4)
Other:
- board text removed: "Boot"
- board text removed: "Reset"
